File: power-supply.kicad_sch (KiCad schematic)
At the start: 9 parts, among them U1 AP62301WU7

Commit message: Add: Board size changes
Parts:
- L1: Int @ 10 1.53 -> (none); MPN XAL5030-222MEC -> (none); Mfr Coilcraft -> (none); SKU 994-XAL5030-222MEC -> (none); Vendor Mouser -> (none)
Changed lines of the file:
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@@
       (effects (font (size 1.27 1.27)) hide)
     )
-    (property "Int @ 10" "1.53" (id 4) (at 175.26 95.25 0)
+    (property "Int @ 10" "" (id 4) (at 175.26 95.25 0)
       (effects (font (size 1.27 1.27)) hide)
     )
-    (property "MPN" "XAL5030-222MEC" (id 5) (at 175.26 95.25 0)
+    (property "MPN" "" (id 5) (at 175.26 95.25 0)
       (effects (font (size 1.27 1.27)) hide)
     )
-    (property "Mfr" "Coilcraft" (id 6) (at 175.26 95.25 0)
+    (property "Mfr" "" (id 6) (at 175.26 95.25 0)
       (effects (font (size 1.27 1.27)) hide)
     )
-    (property "SKU" "994-XAL5030-222MEC" (id 7) (at 175.26 95.25 0)
+    (property "SKU" "" (id 7) (at 175.26 95.25 0)
       (effects (font (size 1.27 1.27)) hide)
     )
-    (property "Vendor" "Mouser" (id 8) (at 175.26 95.25 0)
+    (property "Vendor" "" (id 8) (at 175.26 95.25 0)
       (effects (font (size 1.27 1.27)) hide)
     )

Commit message: Change: Separate boards rather than using mousebites
Parts:
- C1: Int @ 10 0.059 -> 0.062; Stock Situation (none) -> OK @ 2Nov2022
- C19, C3: Int @ 10 0.248 -> 0.174; Stock Situation (none) -> OK @ 2Nov2022
- C2: Int @ 10 0.069 -> 0.038; Stock Situation (none) -> OK @ 2Nov2022
- L1: Int @ 10 (none) -> 2.10; MPN (none) -> XAL5030-222MEC; Mfr (none) -> Coilcraft Ltd.; SKU (none) -> 994-XAL5030-222MEC; Stock Situation (none) -> OK @ 2Nov2022; Vendor (none) -> Mouser
- U1: Int @ 10 0.282 -> 0.366; Stock Situation (none) -> OK @ 2Nov2022
Changed lines of the file:
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@@
       (effects (font (size 1.27 1.27)) hide)
     )
-    (property "Int @ 10" "" (id 4) (at 175.26 95.25 0)
-      (effects (font (size 1.27 1.27)) hide)
-    )
-    (property "MPN" "" (id 5) (at 175.26 95.25 0)
-      (effects (font (size 1.27 1.27)) hide)
-    )
-    (property "Mfr" "" (id 6) (at 175.26 95.25 0)
-      (effects (font (size 1.27 1.27)) hide)
-    )
-    (property "SKU" "" (id 7) (at 175.26 95.25 0)
-      (effects (font (size 1.27 1.27)) hide)
-    )
-    (property "Vendor" "" (id 8) (at 175.26 95.25 0)
+    (property "Int @ 10" "2.10" (id 4) (at 175.26 95.25 0)
+      (effects (font (size 1.27 1.27)) hide)
+    )
+    (property "MPN" "XAL5030-222MEC" (id 5) (at 175.26 95.25 0)
+      (effects (font (size 1.27 1.27)) hide)
+    )
+    (property "Mfr" "Coilcraft Ltd." (id 6) (at 175.26 95.25 0)
+      (effects (font (size 1.27 1.27)) hide)
+    )
+    (property "SKU" "994-XAL5030-222MEC" (id 7) (at 175.26 95.25 0)
+      (effects (font (size 1.27 1.27)) hide)
+    )
+    (property "Vendor" "Mouser" (id 8) (at 175.26 95.25 0)
+      (effects (font (size 1.27 1.27)) hide)
+    )
+    (property "Stock Situation" "OK @ 2Nov2022" (id 9) (at 175.26 95.25 0)
       (effects (font (size 1.27 1.27)) hide)
     )
@@
       (effects (font (size 1.27 1.27)) hide)
     )
-    (property "Int @ 10" "0.248" (id 4) (at 194.31 109.22 0)
+    (property "Int @ 10" "0.174" (id 4) (at 194.31 109.22 0)
       (effects (font (size 1.27 1.27)) hide)
     )
@@
     )
     (property "Vendor" "Mouser" (id 8) (at 194.31 109.22 0)
+      (effects (font (size 1.27 1.27)) hide)
+    )
+    (property "Stock Situation" "OK @ 2Nov2022" (id 9) (at 194.31 109.22 0)
       (effects (font (size 1.27 1.27)) hide)
     )
@@
       (effects (font (size 1.27 1.27)) hide)
     )
-    (property "Int @ 10" "0.282" (id 4) (at 137.16 92.71 0)
+    (property "Int @ 10" "0.366" (id 4) (at 137.16 92.71 0)
       (effects (font (size 1.27 1.27)) hide)
     )
@@
     )
     (property "Vendor" "Mouser" (id 8) (at 137.16 92.71 0)
+      (effects (font (size 1.27 1.27)) hide)
+    )
+    (property "Stock Situation" "OK @ 2Nov2022" (id 9) (at 137.16 92.71 0)
       (effects (font (size 1.27 1.27)) hide)
     )
@@
       (effects (font (size 1.27 1.27)) hide)
     )
-    (property "Int @ 10" "0.069" (id 4) (at 153.67 90.17 0)
+    (property "Int @ 10" "0.038" (id 4) (at 153.67 90.17 0)
       (effects (font (size 1.27 1.27)) hide)
     )
@@
     )
     (property "Vendor" "Mouser" (id 8) (at 153.67 90.17 0)
+      (effects (font (size 1.27 1.27)) hide)
+    )
+    (property "Stock Situation" "OK @ 2Nov2022" (id 9) (at 153.67 90.17 0)
       (effects (font (size 1.27 1.27)) hide)
     )
@@
       (effects (font (size 1.27 1.27)) hide)
     )
-    (property "Int @ 10" "0.248" (id 4) (at 209.55 109.22 0)
+    (property "Int @ 10" "0.174" (id 4) (at 209.55 109.22 0)
       (effects (font (size 1.27 1.27)) hide)
     )
@@
     )
     (property "Vendor" "Mouser" (id 8) (at 209.55 109.22 0)
+      (effects (font (size 1.27 1.27)) hide)
+    )
+    (property "Stock Situation" "OK @ 2Nov2022" (id 9) (at 209.55 109.22 0)
       (effects (font (size 1.27 1.27)) hide)
     )
@@
       (effects (font (size 1.27 1.27)) hide)
     )
-    (property "Int @ 10" "0.059" (id 4) (at 105.41 97.79 0)
+    (property "Int @ 10" "0.062" (id 4) (at 105.41 97.79 0)
       (effects (font (size 1.27 1.27)) hide)
     )
@@
       (effects (font (size 1.27 1.27)) hide)
     )
+    (property "Stock Situation" "OK @ 2Nov2022" (id 9) (at 105.41 97.79 0)
+      (effects (font (size 1.27 1.27)) hide)
+    )
