File: p3-cellular-module.kicad_pcb (KiCad board)
At the start: 4 copper layers, 42 x 55.8 mm, 102 parts, among them J2 SIM8060-6-1-14-00-A, J4 Pogo Pins, Q1 BC818, SW1 KMR221GLFS, U1 AP62301WU7, U2 EG25G, U3 USBLC6-2SC6

Commit message: Change: Separate boards rather than using mousebites
Parts:
- removed the REF** at (141.6, 99.0)
- removed the REF** at (147.6, 99.0)
- removed the REF** at (128.6, 100.8)
- removed the REF** at (132.6, 100.8)
- removed the REF** at (159.6, 100.8)
- removed the REF** at (127.6, 99.0)
- removed the REF** at (132.6, 99.0)
- removed the REF** at (141.6, 100.8)
- removed the REF** at (162.6, 99.0)
- removed the REF** at (142.6, 100.8)
- removed the REF** at (149.6, 99.0)
- removed the REF** at (148.6, 100.8)
- removed the REF** at (139.6, 100.8)
- removed the REF** at (152.6, 100.8)
- removed the REF** at (131.6, 100.8)
- removed the REF** at (161.6, 100.8)
- removed the REF** at (158.6, 99.0)
- removed the REF** at (151.6, 99.0)
- removed the REF** at (140.6, 100.8)
- removed the REF** at (148.6, 99.0)
- removed the REF** at (128.6, 99.0)
- removed the REF** at (140.6, 99.0)
- removed the REF** at (161.6, 99.0)
- removed the REF** at (138.6, 100.8)
- removed the REF** at (131.6, 99.0)
- removed the REF** at (130.6, 100.8)
- removed the REF** at (160.6, 99.0)
- removed the REF** at (129.6, 99.0)
- removed the REF** at (147.6, 100.8)
- removed the REF** at (157.6, 100.8)
- removed the REF** at (138.6, 99.0)
- removed the REF** at (162.6, 100.8)
- removed the REF** at (157.6, 99.0)
- removed the REF** at (139.6, 99.0)
- removed the REF** at (149.6, 100.8)
- removed the REF** at (151.6, 100.8)
- removed the REF** at (159.6, 99.0)
- removed the REF** at (127.6, 100.8)
- removed the REF** at (137.6, 100.8)
- removed the REF** at (150.6, 100.8)
- removed the REF** at (150.6, 99.0)
- removed the REF** at (130.6, 99.0)
- removed the REF** at (137.6, 99.0)
- removed the REF** at (158.6, 100.8)
- removed the REF** at (129.6, 100.8)
- removed the REF** at (152.6, 99.0)
- removed the REF** at (160.6, 100.8)
- removed the REF** at (142.6, 99.0)
- J4: footprint Connector_PinHeader_2.00mm:PinHeader_1x04_P2.00mm_Vertical -> art:PogoPins
- moved J4 3.01 mm to (156.9, 91.5)
Routing:
- net GND: vias 431 -> 438
Other:
- outline, holes or cut-outs redrawn
- board text added: "B"
- board text removed: "A"

Commit message: Add: Gerbers for Rev2
Parts:
- moved J4 0.47 mm to (156.4, 91.5)
Routing:
- net /USB Connector/USB_DP_RAW: track 17.5 -> 16.9 mm
Changed lines of the file:
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@@
   )
   (footprint "art:PogoPins" (layer "F.Cu")
-    (at 156.875 91.45 -90)
+    (at 156.4 91.45 -90)
     (property "Sheetfile" "usb-connector.kicad_sch")
     (property "Sheetname" "USB Connector")
@@
   (segment (start 156.775 137.275) (end 159.125 137.275) (width 0.254) (layer "B.Cu") (net 22))
   (segment (start 159.85 138) (end 160.75 138) (width 0.254) (layer "B.Cu") (net 22))
-  (segment (start 154.59648 90.34648) (end 154.40352 90.15352) (width 0.254) (layer "F.Cu") (net 23))
+  (segment (start 153.95352 90.15352) (end 140.49648 90.15352) (width 0.254) (layer "F.Cu") (net 23))
+  (segment (start 153.882 91.45) (end 153.882 91.239516) (width 0.254) (layer "F.Cu") (net 23))
   (segment (start 140.475 90.175) (end 140.475 90.5) (width 0.254) (layer "F.Cu") (net 23))
-  (segment (start 154.40352 90.15352) (end 140.49648 90.15352) (width 0.254) (layer "F.Cu") (net 23))
-  (segment (start 154.59648 90.90352) (end 154.59648 90.34648) (width 0.254) (layer "F.Cu") (net 23))
   (segment (start 141.15 91.175) (end 141.15 91.7125) (width 0.254) (layer "F.Cu") (net 23))
-  (segment (start 153.882 91.45) (end 154.05 91.45) (width 0.254) (layer "F.Cu") (net 23))
-  (segment (start 140.49648 90.15352) (end 140.475 90.175) (width 0.254) (layer "F.Cu") (net 23))
-  (segment (start 154.05 91.45) (end 154.59648 90.90352) (width 0.254) (layer "F.Cu") (net 23))
+  (segment (start 153.882 91.239516) (end 154.3 90.821516) (width 0.254) (layer "F.Cu") (net 23))
+  (segment (start 154.3 90.821516) (end 154.3 90.5) (width 0.254) (layer "F.Cu") (net 23))
+  (segment (start 154.3 90.5) (end 153.95352 90.15352) (width 0.254) (layer "F.Cu") (net 23))
   (segment (start 140.475 90.5) (end 141.15 91.175) (width 0.254) (layer "F.Cu") (net 23))
+  (segment (start 140.49648 90.15352) (end 140.475 90.175) (width 0.254) (layer "F.Cu") (net 23))
   (segment (start 143.537298 111.837298) (end 147.304807 115.604807) (width 0.254) (layer "F.Cu") (net 24))
   (segment (start 142.7 94.8) (end 142.7 96.2) (width 0.254) (layer "F.Cu") (net 24))
   (segment (start 143.9985 103.2) (end 143.828531 103.369969) (width 0.254) (layer "F.Cu") (net 24))
   (segment (start 141.15 93.9875) (end 141.8875 93.9875) (width 0.254) (layer "F.Cu") (net 24))
-  (segment (start 148.71902 116.190593) (end 149.139943 116.190593) (width 0.254) (layer "F.Cu") (net 24))
+  (segment (start 148.929481 116.190593) (end 148.71902 116.190593) (width 0.254) (layer "F.Cu") (net 24))
   (segment (start 143.828531 103.369969) (end 143.330635 103.369969) (width 0.254) (layer "F.Cu") (net 24))
-  (segment (start 149.799675 116.850325) (end 149.139943 116.190593) (width 0.254) (layer "F.Cu") (net 24))
+  (segment (start 149.288761 116.339411) (end 149.799675 116.850325) (width 0.254) (layer "F.Cu") (net 24))
   (segment (start 142.951511 104.163307) (end 142.951511 110.423084) (width 0.254) (layer "F.Cu") (net 24))
   (segment (start 143.330635 103.369969) (end 143.244404 103.4562) (width 0.254) (layer "F.Cu") (net 24))
@@
   (arc (start 148.71902 116.190593) (mid 147.953653 116.038352) (end 147.304807 115.604807) (width 0.254) (layer "F.Cu") (net 24))
   (arc (start 142.951511 110.423084) (mid 143.103752 111.188451) (end 143.537298 111.837298) (width 0.254) (layer "F.Cu") (net 24))
+  (arc (start 149.288761 116.339411) (mid 149.123922 116.229269) (end 148.929481 116.190593) (width 0.254) (layer "F.Cu") (net 24))
   (segment (start 150.7 116.45) (end 150.7 115.577454) (width 0.254) (layer "B.Cu") (net 24))
   (segment (start 149.799675 116.850325) (end 150.299675 116.850325) (width 0.254) (layer "B.Cu") (net 24))
   (segment (start 150.299675 116.850325) (end 150.7 116.45) (width 0.254) (layer "B.Cu") (net 24))
-  (segment (start 140.175 89.7) (end 140 89.875) (width 0.254) (layer "F.Cu") (net 25))
-  (segment (start 154.625 89.7) (end 140.175 89.7) (width 0.254) (layer "F.Cu") (net 25))
-  (segment (start 155.882 90.957) (end 154.625 89.7) (width 0.254) (layer "F.Cu") (net 25))
-  (segment (start 155.882 91.45) (end 155.882 90.957) (width 0.254) (layer "F.Cu") (net 25))
-  (segment (start 140 89.875) (end 140 90.5) (width 0.254) (layer "F.Cu") (net 25))
   (segment (start 139.25 91.25) (end 139.25 91.7125) (width 0.254) (layer "F.Cu") (net 25))
+  (segment (start 155.882 91.45) (end 155.882 91.382) (width 0.254) (layer "F.Cu") (net 25))
+  (segment (start 140 89.875) (end 140 90.5) (width 0.254) (layer "F.Cu") (net 25))
+  (segment (start 154.2 89.7) (end 140.175 89.7) (width 0.254) (layer "F.Cu") (net 25))
   (segment (start 140 90.5) (end 139.25 91.25) (width 0.254) (layer "F.Cu") (net 25))
+  (segment (start 140.175 89.7) (end 140 89.875) (width 0.254) (layer "F.Cu") (net 25))
+  (segment (start 155.882 91.382) (end 154.2 89.7) (width 0.254) (layer "F.Cu") (net 25))
   (segment (start 143.405031 104.01979) (end 143.405031 110.23523) (width 0.254) (layer "F.Cu") (net 26))
   (segment (start 143.990818 111.649444) (end 147.452068 115.110694) (width 0.254) (layer "F.Cu") (net 26))
-  (segment (start 150.65 116.849984) (end 150.65 116.85) (width 0.254) (layer "F.Cu") (net 26))
-  (segment (start 149.942099 116.142083) (end 150.65 116.849984) (width 0.254) (layer "F.Cu") (net 26))
+  (segment (start 149.942099 116.142083) (end 149.942083 116.142083) (width 0.254) (layer "F.Cu") (net 26))
+  (segment (start 150.974258 116.85) (end 151.2985 116.85) (width 0.254) (layer "F.Cu") (net 26))
   (segment (start 144 102.4) (end 144.2 102.6) (width 0.254) (layer "F.Cu") (net 26))
-  (segment (start 149.942083 116.142083) (end 149.942099 116.142083) (width 0.254) (layer "F.Cu") (net 26))
   (segment (start 139.25 95.1) (end 139.3 95.15) (width 0.254) (layer "F.Cu") (net 26))
   (segment (start 144.453553 103.678554) (end 144.385089 103.747018) (width 0.254) (layer "F.Cu") (net 26))
@@
   (segment (start 144.6 102.799999) (end 144.6 103.325) (width 0.254) (layer "F.Cu") (net 26))
   (segment (start 144.4 102.6) (end 144.2 102.6) (width 0.254) (layer "F.Cu") (net 26))
-  (segment (start 150.65 116.85) (end 151.2985 116.85) (width 0.254) (layer "F.Cu") (net 26))
+  (segment (start 150.420742 116.620726) (end 149.942099 116.142083) (width 0.254) (layer "F.Cu") (net 26))
   (segment (start 139.25 93.9875) (end 139.25 95.1) (width 0.254) (layer "F.Cu") (net 26))
   (segment (start 143.518489 103.823489) (end 143.463609 103.878369) (width 0.254) (layer "F.Cu") (net 26))
@@
   (arc (start 143.405031 104.01979) (mid 143.420255 103.943254) (end 143.463609 103.878369) (width 0.254) (layer "F.Cu") (net 26))
   (arc (start 143.405031 110.23523) (mid 143.557272 111.000597) (end 143.990818 111.649444) (width 0.254) (layer "F.Cu") (net 26))
+  (arc (start 150.420742 116.620726) (mid 150.674697 116.790413) (end 150.974258 116.85) (width 0.254) (layer "F.Cu") (net 26))
   (arc (start 144.6 102.799999) (mid 144.541421 102.658578) (end 144.4 102.6) (width 0.254) (layer "F.Cu") (net 26))
   (arc (start 148.866281 115.69648) (mid 148.100914 115.544239) (end 147.452068 115.110694) (width 0.254) (layer "F.Cu") (net 26))
@@
   (zone (net 8) (net_name "/Cellular Modem/USIM_VDD") (layers "F.Cu" "In1.Cu") (hatch edge 0.508)
     (priority 10)
-    (connect_pads yes (clearance 0.1))
+    (connect_pads yes (clearance 0))
     (min_thickness 0.254) (filled_areas_thickness no)
     (fill yes (thermal_gap 0.508) (thermal_bridge_width 0.508))
